File: ArquivosEagle/LabDuino/LabDuino.sch (EAGLE design)
At the start: 40 parts, among them IC1 PCF8574P, IC2 PCF8574P

Commit message: Board Update
Parts:
- added R14: (no value), SparkFun-Resistors:RESISTORPTH-1/6W
- R5: device pot:TRIM_US-B25P -> pot:TRIM_US-RS3
Connections:
- new net N$27: DIS1.NC@1, R14.2
- net GND: now also R5.E; no longer R5.S
- net N$14: now also R5.S; no longer R5.E
- net VCC: now also R14.1; no longer DIS1.NC@1
Other:
- moved on the sheet: C2, R5
Changed lines of the file:
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@@
 </variantdefs>
 <classes>
-<class number="0" name="default" width="1.5" drill="0.254">
-<clearance class="0" value="2"/>
+<class number="0" name="default" width="0.254" drill="0.381">
+<clearance class="0" value="0.508"/>
 </class>
 </classes>
@@
 <part name="SUPPLY14" library="supply2" deviceset="GND" device=""/>
 <part name="DIS1" library="display-lcd" deviceset="TUXGR_16X2_R2" device=""/>
-<part name="SUPPLY15" library="supply2" deviceset="VCC" device=""/>
 <part name="SUPPLY16" library="supply2" deviceset="GND" device=""/>
 <part name="SUPPLY17" library="supply2" deviceset="GND" device=""/>
-<part name="R5" library="pot" deviceset="TRIM_US-" device="B25P"/>
-<part name="SUPPLY19" library="supply2" deviceset="GND" device=""/>
 <part name="D1" library="diode" deviceset="1N4004" device=""/>
 <part name="S1" library="switch" deviceset="TL32PO" device=""/>
@@
 <part name="SUPPLY21" library="supply2" deviceset="GND" device=""/>
 <part name="SUPPLY22" library="supply2" deviceset="GND" device=""/>
-<part name="P+1" library="supply1" deviceset="VCC" device=""/>
 <part name="P+2" library="supply1" deviceset="VCC" device=""/>
 <part name="P+3" library="supply1" deviceset="VCC" device=""/>
 <part name="P+4" library="supply1" deviceset="VCC" device=""/>
 <part name="P+5" library="supply1" deviceset="VCC" device=""/>
-<part name="P+8" library="supply1" deviceset="VCC" device=""/>
 <part name="R6" library="resistor" deviceset="R-US_" device="0204/7"/>
 <part name="R7" library="resistor" deviceset="R-US_" device="0204/7"/>
@@
 <part name="SE-" library="wirepad" deviceset="1,6/0,9" device=""/>
 <part name="SUPPLY1" library="supply2" deviceset="GND" device=""/>
+<part name="P+11" library="supply1" deviceset="VCC" device=""/>
+<part name="R14" library="SparkFun-Resistors" deviceset="RESISTOR" device="PTH-1/6W"/>
+<part name="P+1" library="supply1" deviceset="VCC" device=""/>
+<part name="R5" library="pot" deviceset="TRIM_US-" device="RS3"/>
+<part name="P+8" library="supply1" deviceset="VCC" device=""/>
+<part name="SUPPLY9" library="supply2" deviceset="GND" device=""/>
 </parts>
 <sheets>
@@
 <instance part="SUPPLY14" gate="GND" x="30.48" y="50.8" rot="R90"/>
 <instance part="DIS1" gate="G$1" x="-10.16" y="78.74"/>
-<instance part="SUPPLY15" gate="G$1" x="-25.4" y="66.04" rot="R180"/>
 <instance part="SUPPLY16" gate="GND" x="-27.94" y="66.04"/>
-<instance part="SUPPLY17" gate="GND" x="10.16" y="66.04"/>
-<instance part="R5" gate="G$1" x="-22.86" y="40.64"/>
-<instance part="SUPPLY19" gate="GND" x="-17.78" y="38.1"/>
+<instance part="SUPPLY17" gate="GND" x="17.78" y="71.12" rot="R180"/>
 <instance part="D1" gate="1" x="119.38" y="15.24"/>
 <instance part="S1" gate="BEF1" x="104.14" y="10.16"/>
@@
 <instance part="SUPPLY27" gate="GND" x="33.02" y="66.04"/>
 <instance part="C1" gate="G$1" x="127" y="12.7"/>
-<instance part="C2" gate="G$1" x="147.32" y="12.7"/>
+<instance part="C2" gate="G$1" x="149.86" y="12.7"/>
 <instance part="SUPPLY21" gate="GND" x="127" y="5.08"/>
-<instance part="SUPPLY22" gate="GND" x="147.32" y="5.08"/>
-<instance part="P+1" gate="VCC" x="7.62" y="66.04" rot="R180"/>
+<instance part="SUPPLY22" gate="GND" x="149.86" y="5.08"/>
 <instance part="P+2" gate="VCC" x="2.54" y="27.94" rot="R90"/>
 <instance part="P+3" gate="VCC" x="30.48" y="10.16" rot="R270"/>
 <instance part="P+4" gate="VCC" x="33.02" y="93.98"/>
 <instance part="P+5" gate="VCC" x="2.54" y="-7.62" rot="R90"/>
-<instance part="P+8" gate="VCC" x="-22.86" y="30.48" rot="R180"/>
 <instance part="R6" gate="G$1" x="30.48" y="99.06"/>
 <instance part="R7" gate="G$1" x="33.02" y="106.68" rot="R180"/>
@@
 <instance part="VCC-BT" gate="1" x="-55.88" y="25.4" rot="R90"/>
 <instance part="P+7" gate="VCC" x="-53.34" y="27.94" rot="R270"/>
-<instance part="P+6" gate="VCC" x="154.94" y="15.24" rot="R270"/>
+<instance part="P+6" gate="VCC" x="160.02" y="15.24" rot="R270"/>
 <instance part="R10" gate="G$1" x="48.26" y="63.5" rot="R180"/>
 <instance part="R11" gate="G$1" x="45.72" y="58.42" rot="R180"/>
@@
 <instance part="SE-" gate="1" x="66.04" y="104.14" rot="R90"/>
 <instance part="SUPPLY1" gate="GND" x="68.58" y="106.68" rot="R90"/>
+<instance part="P+11" gate="VCC" x="-25.4" y="66.04" rot="R180"/>
+<instance part="R14" gate="G$1" x="12.7" y="63.5" rot="R180"/>
+<instance part="P+1" gate="VCC" x="20.32" y="63.5" rot="R270"/>
+<instance part="R5" gate="G$1" x="-27.94" y="48.26"/>
+<instance part="P+8" gate="VCC" x="-27.94" y="38.1" rot="R180"/>
+<instance part="SUPPLY9" gate="GND" x="-27.94" y="58.42" rot="R180"/>
 </instances>
 <busses>
@@
 <pinref part="DIS1" gate="G$1" pin="NC@2"/>
 <pinref part="SUPPLY17" gate="GND" pin="GND"/>
-</segment>
-<segment>
-<pinref part="R5" gate="G$1" pin="S"/>
-<pinref part="SUPPLY19" gate="GND" pin="GND"/>
+<wire x1="17.78" y1="68.58" x2="10.16" y2="68.58" width="0.1524" layer="91"/>
 </segment>
 <segment>
@@
 <pinref part="SE-" gate="1" pin="P"/>
 <pinref part="SUPPLY1" gate="GND" pin="GND"/>
+</segment>
+<segment>
+<pinref part="R5" gate="G$1" pin="E"/>
+<pinref part="SUPPLY9" gate="GND" pin="GND"/>
 </segment>
 </net>
@@
 <net name="VCC" class="0">
 <segment>
-<pinref part="DIS1" gate="G$1" pin="VCC"/>
-<pinref part="SUPPLY15" gate="G$1" pin="VCC"/>
-</segment>
-<segment>
-<pinref part="DIS1" gate="G$1" pin="NC@1"/>
-<pinref part="P+1" gate="VCC" pin="VCC"/>
-</segment>
-<segment>
 <pinref part="IC1" gate="G$1" pin="VDD"/>
 <pinref part="P+2" gate="VCC" pin="VCC"/>
@@
 </segment>
 <segment>
+<pinref part="VCC-BT" gate="1" pin="P"/>
+<pinref part="P+7" gate="VCC" pin="VCC"/>
+</segment>
+<segment>
+<pinref part="C2" gate="G$1" pin="+"/>
+<pinref part="P+6" gate="VCC" pin="VCC"/>
+<wire x1="157.48" y1="15.24" x2="149.86" y2="15.24" width="0.1524" layer="91"/>
+<pinref part="IC4" gate="G$1" pin="OUT"/>
+<wire x1="144.78" y1="15.24" x2="149.86" y2="15.24" width="0.1524" layer="91"/>
+<junction x="149.86" y="15.24"/>
+</segment>
+<segment>
+<pinref part="VCC-DG" gate="1" pin="P"/>
+<pinref part="P+9" gate="VCC" pin="VCC"/>
+</segment>
+<segment>
+<pinref part="P+10" gate="VCC" pin="VCC"/>
+<pinref part="SE+" gate="1" pin="P"/>
+</segment>
+<segment>
+<pinref part="DIS1" gate="G$1" pin="VCC"/>
+<pinref part="P+11" gate="VCC" pin="VCC"/>
+</segment>
+<segment>
+<pinref part="R14" gate="G$1" pin="1"/>
+<pinref part="P+1" gate="VCC" pin="VCC"/>
+</segment>
+<segment>
 <pinref part="R5" gate="G$1" pin="A"/>
 <pinref part="P+8" gate="VCC" pin="VCC"/>
-</segment>
-<segment>
-<pinref part="VCC-BT" gate="1" pin="P"/>
-<pinref part="P+7" gate="VCC" pin="VCC"/>
-</segment>
-<segment>
-<pinref part="C2" gate="G$1" pin="+"/>
-<pinref part="P+6" gate="VCC" pin="VCC"/>
-<wire x1="152.4" y1="15.24" x2="147.32" y2="15.24" width="0.1524" layer="91"/>
-<pinref part="IC4" gate="G$1" pin="OUT"/>
-<wire x1="144.78" y1="15.24" x2="147.32" y2="15.24" width="0.1524" layer="91"/>
-</segment>
-<segment>
-<pinref part="VCC-DG" gate="1" pin="P"/>
-<pinref part="P+9" gate="VCC" pin="VCC"/>
-</segment>
-<segment>
-<pinref part="P+10" gate="VCC" pin="VCC"/>
-<pinref part="SE+" gate="1" pin="P"/>
 </segment>
 </net>
@@
 <pinref part="DIS1" gate="G$1" pin="CONTR"/>
 <wire x1="-22.86" y1="68.58" x2="-22.86" y2="48.26" width="0.1524" layer="91"/>
-<pinref part="R5" gate="G$1" pin="E"/>
+<pinref part="R5" gate="G$1" pin="S"/>
 </segment>
 </net>
@@
 </segment>
 </net>
+<net name="N$27" class="0">
+<segment>
+<pinref part="DIS1" gate="G$1" pin="NC@1"/>
+<pinref part="R14" gate="G$1" pin="2"/>
+<wire x1="7.62" y1="68.58" x2="7.62" y2="63.5" width="0.1524" layer="91"/>
+</segment>
+</net>
